File: FE_4CH/HW/v3.0/v3.0.kicad_sch (KiCad schematic)
At the start: 158 parts, among them J1 SMA-ANG, J2 PINH_2MM_2P, J3 USB4080-03-A, J6 MS300-10F, U1 MAX2771, U10 74AVC9112DCH, U11 PI3USB302-AZBEX, U2 MAX2771, U3 MAX2771, U4 MAX2771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

Commit message: replace wilkinson splitter with double, add mounting holes and fidushes
Parts:
- added FID1, FID2, FID3: Fiducial, Fiducial:Fiducial_0.75mm_Mask1.5mm, symbol Mechanical:Fiducial
- added H1, H2, H3, H4: MountingHole_Pad, MountingHole:MountingHole_2.2mm_M2_DIN965_Pad, symbol Mechanical:MountingHole_Pad
- added R23, R24, R25: 100, pocket_sdr_v2.3:C1005, symbol pocket_sdr_v2.3-eagle-import:R1005
- R1, R2, R3: value 100 -> 200
- RD1, RD2, RD3: value PD0922J5050S2HF -> PD0922J5050D2HF
Connections:
- net GND: now also H1.1, H2.1, H3.1, H4.1; no longer RD1.1 (GND@1), RD1.3 (GND@2), RD2.1 (GND@1), RD2.3 (GND@2), RD3.1 (GND@1), RD3.3 (GND@2)
- net at R2.2 (P$2), RS1.5 (RFIN): now also RD2.1 (OUT2); no longer RD2.6 (OUT2)
- net at R1.1 (P$1), RD3.2 (INPUT): now also RD1.6 (OUT1); no longer RD1.4 (OUT1)
- net at R1.2 (P$2), RD2.2 (INPUT): now also RD1.1 (OUT2); no longer RD1.6 (OUT2)
- net at R3.1 (P$1), RS4.5 (RFIN): now also RD3.6 (OUT1); no longer RD3.4 (OUT1)
- net at R3.2 (P$2), RS3.5 (RFIN): now also RD3.1 (OUT2); no longer RD3.6 (OUT2)
- net at R2.1 (P$1), RS2.5 (RFIN): now also RD2.6 (OUT1); no longer RD2.4 (OUT1)
- new net: R23.1 (P$1), RD1.3 (mid2)
- new net: R23.2 (P$2), RD1.4 (mid1)
- new net: R25.1 (P$1), RD3.3 (mid2)
- new net: R25.2 (P$2), RD3.4 (mid1)
- new net: R24.1 (P$1), RD2.3 (mid2)
- new net: R24.2 (P$2), RD2.4 (mid1)
Other:
- moved on the sheet: C2
